File: modules/mult/kicad/mult.kicad_pcb (KiCad board)
At the start: 2 copper layers, 28 x 108 mm, 13 parts, among them J1 Thonkiconn, J10 Thonkiconn, J11 Thonkiconn, J12 Thonkiconn, J2 Thonkiconn, J3 Thonkiconn, J4 Thonkiconn, J5 Thonkiconn, J6 Thonkiconn, J7 Thonkiconn, J8 Thonkiconn, J9 Thonkiconn

Commit message: M1-M3: reject invalid designs, forbid vias in pads, fail closed on export
Three of the roadmap's review findings become code and tests. Every design
is now validated before emission, the router's result is checked on the
final geometry rather than trusted, and nothing can be exported that a
clean check did not produce.

Validation (toolkit/src/Validate.hs, wired into pcbgen before emission):
unique references and net names, every (ref, pin) must exist on the library
symbol, every symbol pin must be on exactly one net or listed in the new
partNoConnect, assembly class and LCSC field must agree, dimensions and
routing settings must be positive. On any diagnostic pcbgen prints them and
exits 1 without writing a file. The four wiring faults ERC used to accept
(U1.8 removed, mistyped as U1.88, on both rails, D2.1 dropped) are rejected
with diagnostics that name the pin.

Routing (toolkit/src/Route/Check.hs, Router.hs): a via may no longer be
placed in or against any pad, its own net included, which is what put 0.3 mm
drills in four SMD solder lands. Pre-routed copper is treated as one terminal
per island, so a hand-drawn trace can no longer make a net look finished
while a pad hangs unconnected, and it now blocks by its own width. Per-net
connectivity and via/pad clearance are recomputed on the emitted geometry;
any failure, contested cell or disconnect aborts generation.

Pours: Zone gains an explicit PadConnect. The attenuverter routes GND as
copper, so its pours no longer bond to pads at all, which also removes the
starved-thermal violation the stricter routing exposed. The mult's sleeves
are held by its pours alone and keep thermal relief; validation rejects an
unbonded pour on a net nothing routes.

Scripts: check.sh writes build/check.ok (tool versions, git provenance,
sha256 of every source and of the zone-filled board) only when ERC and DRC
are both clean, and removes stale copies first. fab.sh refuses unless every
hash still matches, builds into a temporary dire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
Routing:
- net /MULT_A: track 80.3 -> 79.4 mm
- net /MULT_B: track 79.3 -> 80.3 mm
Changed lines of the file:
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@@
 	(segment
 		(start 6.5 44.85)
-		(end 7.3 45.5)
-		(width 0.5)
-		(layer "B.Cu")
-		(net "/MULT_A")
-	)
-	(segment
-		(start 7.3 45.5)
-		(end 7.7 45.7)
-		(width 0.5)
-		(layer "B.Cu")
-		(net "/MULT_A")
-	)
-	(segment
-		(start 7.7 45.7)
-		(end 7.9 45.9)
-		(width 0.5)
-		(layer "B.Cu")
-		(net "/MULT_A")
-	)
-	(segment
-		(start 7.9 45.9)
-		(end 8.1 46.3)
-		(width 0.5)
-		(layer "B.Cu")
-		(net "/MULT_A")
-	)
-	(segment
-		(start 8.1 46.3)
-		(end 8.1 52.1)
-		(width 0.5)
-		(layer "B.Cu")
-		(net "/MULT_A")
-	)
-	(segment
-		(start 8.1 52.1)
-		(end 7.1 57.7)
-		(width 0.5)
-		(layer "B.Cu")
-		(net "/MULT_A")
-	)
-	(segment
-		(start 7.1 57.7)
+		(end 5.7 45.5)
+		(width 0.5)
+		(layer "B.Cu")
+		(net "/MULT_A")
+	)
+	(segment
+		(start 5.7 45.5)
+		(end 5.3 45.7)
+		(width 0.5)
+		(layer "B.Cu")
+		(net "/MULT_A")
+	)
+	(segment
+		(start 5.3 45.7)
+		(end 5.1 45.9)
+		(width 0.5)
+		(layer "B.Cu")
+		(net "/MULT_A")
+	)
+	(segment
+		(start 5.1 45.9)
+		(end 4.9 46.3)
+		(width 0.5)
+		(layer "B.Cu")
+		(net "/MULT_A")
+	)
+	(segment
+		(start 4.9 46.3)
+		(end 4.9 51.9)
+		(width 0.5)
+		(layer "B.Cu")
+		(net "/MULT_A")
+	)
+	(segment
+		(start 4.9 51.9)
+		(end 5.9 57.7)
+		(width 0.5)
+		(layer "B.Cu")
+		(net "/MULT_A")
+	)
+	(segment
+		(start 5.9 57.7)
 		(end 6.5 58.55)
 		(width 0.5)
@@
 	(segment
 		(start 6.5 58.55)
-		(end 7.5 58.3)
-		(width 0.5)
-		(layer "B.Cu")
-		(net "/MULT_A")
-	)
-	(segment
-		(start 7.5 58.3)
-		(end 12.9 58.3)
-		(width 0.5)
-		(layer "B.Cu")
-		(net "/MULT_A")
-	)
-	(segment
-		(start 12.9 58.3)
+		(end 7.5 58.9)
+		(width 0.5)
+		(layer "B.Cu")
+		(net "/MULT_A")
+	)
+	(segment
+		(start 7.5 58.9)
+		(end 8.1 58.9)
+		(width 0.5)
+		(layer "B.Cu")
+		(net "/MULT_A")
+	)
+	(segment
+		(start 8.1 58.9)
+		(end 12.9 58.9)
+		(width 0.5)
+		(layer "B.Cu")
+		(net "/MULT_A")
+	)
+	(segment
+		(start 12.9 58.9)
 		(end 13.35 58.55)
 		(width 0.5)
@@
 	)
 	(segment
-		(start 6.5 58.55)
-		(end 7.3 59.1)
-		(width 0.5)
-		(layer "B.Cu")
-		(net "/MULT_A")
-	)
-	(segment
-		(start 7.3 59.1)
-		(end 8.1 59.9)
-		(width 0.5)
-		(layer "B.Cu")
-		(net "/MULT_A")
-	)
-	(segment
-		(start 8.1 59.9)
-		(end 8.1 64.7)
-		(width 0.5)
-		(layer "B.Cu")
-		(net "/MULT_A")
-	)
-	(segment
-		(start 8.1 64.7)
+		(start 8.1 58.9)
+		(end 8.1 65.7)
+		(width 0.5)
+		(layer "B.Cu")
+		(net "/MULT_A")
+	)
+	(segment
+		(start 8.1 65.7)
 		(end 6.9 71.3)
 		(width 0.5)
@@
 	(segment
 		(start 6.5 85.95)
-		(end 7.3 86.5)
-		(width 0.5)
-		(layer "B.Cu")
-		(net "/MULT_A")
-	)
-	(segment
-		(start 7.3 86.5)
-		(end 8.1 87.3)
-		(width 0.5)
-		(layer "B.Cu")
-		(net "/MULT_A")
-	)
-	(segment
-		(start 8.1 87.3)
-		(end 8.1 92.1)
-		(width 0.5)
-		(layer "B.Cu")
-		(net "/MULT_A")
-	)
-	(segment
-		(start 8.1 92.1)
-		(end 6.9 98.7)
-		(width 0.5)
-		(layer "B.Cu")
-		(net "/MULT_A")
-	)
-	(segment
-		(start 6.9 98.7)
+		(end 5.7 86.5)
+		(width 0.5)
+		(layer "B.Cu")
+		(net "/MULT_A")
+	)
+	(segment
+		(start 5.7 86.5)
+		(end 4.9 87.3)
+		(width 0.5)
+		(layer "B.Cu")
+		(net "/MULT_A")
+	)
+	(segment
+		(start 4.9 87.3)
+		(end 4.9 92.5)
+		(width 0.5)
+		(layer "B.Cu")
+		(net "/MULT_A")
+	)
+	(segment
+		(start 4.9 92.5)
+		(end 6.1 98.7)
+		(width 0.5)
+		(layer "B.Cu")
+		(net "/MULT_A")
+	)
+	(segment
+		(start 6.1 98.7)
 		(end 6.5 99.65)
 		(width 0.5)
@@
 	(segment
 		(start 21.5 58.55)
-		(end 20.5 58.9)
-		(width 0.5)
-		(layer "B.Cu")
-		(net "/MULT_B")
-	)
-	(segment
-		(start 20.5 58.9)
-		(end 19.9 58.9)
-		(width 0.5)
-		(layer "B.Cu")
-		(net "/MULT_B")
-	)
-	(segment
-		(start 19.9 58.9)
-		(end 15.1 58.9)
-		(width 0.5)
-		(layer "B.Cu")
-		(net "/MULT_B")
-	)
-	(segment
-		(start 15.1 58.9)
+		(end 20.5 58.7)
+		(width 0.5)
+		(layer "B.Cu")
+		(net "/MULT_B")
+	)
+	(segment
+		(start 20.5 58.7)
+		(end 15.1 58.7)
+		(width 0.5)
+		(layer "B.Cu")
+		(net "/MULT_B")
+	)
+	(segment
+		(start 15.1 58.7)
 		(end 14.65 58.55)
 		(width 0.5)
@@
 	)
 	(segment
-		(start 19.9 58.9)
-		(end 19.9 65.5)
-		(width 0.5)
-		(layer "B.Cu")
-		(net "/MULT_B")
-	)
-	(segment
-		(start 19.9 65.5)
+		(start 21.5 58.55)
+		(end 20.7 59.1)
+		(width 0.5)
+		(layer "B.Cu")
+		(net "/MULT_B")
+	)
+	(segment
+		(start 20.7 59.1)
+		(end 19.9 59.9)
+		(width 0.5)
+		(layer "B.Cu")
+		(net "/MULT_B")
+	)
+	(segment
+		(start 19.9 59.9)
+		(end 19.9 64.9)
+		(width 0.5)
+		(layer "B.Cu")
+		(net "/MULT_B")
+	)
+	(segment
+		(start 19.9 64.9)
 		(end 21.1 71.3)
 		(width 0.5)
@@
 	(segment
 		(start 19.9 73.7)
-		(end 19.9 78.3)
-		(width 0.5)
-		(layer "B.Cu")
-		(net "/MULT_B")
-	)
-	(segment
-		(start 19.9 78.3)
+		(end 19.9 78.9)
+		(width 0.5)
+		(layer "B.Cu")
+		(net "/MULT_B")
+	)
+	(segment
+		(start 19.9 78.9)
 		(end 20.9 85.1)
 		(width 0.5)
