File: modules/mult/kicad/mult.kicad_pcb (KiCad board)
At the start: 2 copper layers, 28 x 108 mm, 13 parts, among them J1 Thonkiconn, J10 Thonkiconn, J11 Thonkiconn, J12 Thonkiconn, J2 Thonkiconn, J3 Thonkiconn, J4 Thonkiconn, J5 Thonkiconn, J6 Thonkiconn, J7 Thonkiconn, J8 Thonkiconn, J9 Thonkiconn

Commit message: Attenuverter option B: precision circuit, models, eight decks, 100 mm boards
The attenuverter becomes the option B design the user chose: one OPA2197
per channel as unity-gain input buffer plus attenuverter stage, 10k 0.1%
thin-film gain resistors with 10 pF C0G compensation, a 1M input and a
REF5050 offset reference. OPA2197 and REF5050 models are built from the
datasheet maxima with input capacitance, a second pole and TEMPER terms.
Emit.Spice learns Reference_Voltage symbols and places a 0 V probe in every
op-amp output so a deck can measure loop gain by voltage injection on the
generated netlist. Eight decks assert every limit in the error budget and
pass: the stage has 72 degrees of phase margin with the capacitor and 27
without; the gain resistors are 10k rather than the assumed 100k because
the input capacitance shelved the full-clockwise response 4.6 % at 20 kHz
with 100k. eurorackPcbHeight drops to 100 mm for every module; the
attenuverter's SMD moves into the pad-free strips between its controls.
65 tests, both pipelines and sim.sh pass; the decision file is retired
into SPEC.md.

Co-Authored-By: Claude Fable 5.1 <noreply@anthropic.com>
Parts:
- moved J2 4.00 mm to (6.50, 29.4)
- moved J8 4.00 mm to (21.5, 29.4)
- moved J1 4.00 mm to (6.50, 15.8)
- moved J10 4.00 mm to (21.5, 56.9)
- moved J11 4.00 mm to (21.5, 70.5)
- moved J12 4.00 mm to (21.5, 84.2)
- moved J3 4.00 mm to (6.50, 43.1)
- moved J4 4.00 mm to (6.50, 56.9)
- moved J5 4.00 mm to (6.50, 70.5)
- moved J6 4.00 mm to (6.50, 84.2)
- moved J7 4.00 mm to (21.5, 15.8)
- moved J9 4.00 mm to (21.5, 43.1)
- moved JP1 4.00 mm to (14.0, 54.5)
Other:
- board size 28 x 108 mm -> 28 x 100 mm
